Commit message: fixed paths

File: urdf/prarob_manipulator.urdf.xacro (robot description, xacro)
@@ -1,6 +1,6 @@
 <?xml version="1.0"?>
 <robot name="prarob_manipulator" xmlns:xacro="http://ros.org/wiki/xacro">
-  <xacro:include filename="$(find ros2_prarob)/urdf/prarob_manipulator.xacro" />
-  <xacro:include filename="$(find ros2_prarob)/urdf/prarob_manipulator.ros2_control.xacro" />
+  <xacro:include filename="$(find connect_the_bdots)/urdf/prarob_manipulator.xacro" />
+  <xacro:include filename="$(find connect_the_bdots)/urdf/prarob_manipulator.ros2_control.xacro" />
   <link name="world"/>
   <xacro:prarob_manipulator parent="world">

File: urdf/prarob_manipulator.xacro (robot description, xacro)
@@ -30,5 +30,5 @@
       <origin rpy="0 0 0" xyz="0 0 0"/>
       <geometry>
-        <mesh filename="package://ros2_prarob/meshes/postolje_seminar_v1.stl" scale="0.01 0.01 0.01"/>
+        <mesh filename="package://connect_the_bdots/meshes/SeminarBase.step" scale="0.01 0.01 0.01"/>
       </geometry>
       <material name="">
@@ -39,5 +39,5 @@
       <origin rpy="0 0 0" xyz="0 0 0"/>
       <geometry>
-        <mesh filename="package://ros2_prarob/meshes/postolje_seminar_v1.stl" scale="0.01 0.01 0.01"/>
+        <mesh filename="package://connect_the_bdots/meshes/SeminarBase.step" scale="0.01 0.01 0.01"/>
       </geometry>
     </collision>
